File: PCB/Main Boards/OSO-JOLT-A1/OSO-JOLT-A1.kicad_sch (KiCad schematic)
At the start: 34 parts, among them J1 OSO_SWD, J2 FH19C-9S-0.5SH_10_, Q1 Q_NMOS_GSD, U1 ATSAML22J18A-MUT, U4 MIC5365-3.3YC5-TR, X1 Crystal

Commit message: Removed the daughterboard connector and placed LIS2DW directly on board
Parts:
- removed J2: FH19C-9S-0.5SH_10_, OSO-SWAT-A1-05:FH19C9S05SH10, symbol OSO-SWAT-A1-05-eagle-import:FH19C-9S-0.5SH_10_
- added C10: 10uF, Capacitor_SMD:C_0603_1608Metric, symbol OSO-SWAT-A1-05-eagle-import:CAP_CERAMIC_0603MP
- added C11: 0.1uF, Capacitor_SMD:C_0603_1608Metric, symbol OSO-SWAT-A1-05-eagle-import:CAP_CERAMIC_0603MP
- added U6: LIS2DW12TR, OSO-SWAT-A1-05:LGA12R50P4X4_200X200X70, symbol OSO-SWD:LIS2DW12TR
Connections:
- net A3/D0/CS: now also U6.11 (INT2)
- net A4/D1/MISO: now also U6.12 (INT1)
- net GND: now also C10.2, C11.2, U6.6 (GND), U6.7 (RES), U6.8 (GND)
- net SCL: now also U6.1 (SCL/SPC)
- net SDA: now also U6.4 (SDA/SDI/SDO)
- net VCC: now also C10.1, C11.1, U6.10 (VDD_IO), U6.2 (CS), U6.3 (SDO/SDA0), U6.9 (VDD)
- no-connect marks 9 -> 10
Other:
- note removed: "--LOCKED--"
- moved on the sheet: D2, R2, R3, R4, R5, R6

Commit message: This commit is what holds the design sent to JLCPCB
Parts:
- added Q2: Q_Photo_NPN, Resistor_SMD:R_0603_1608Metric, symbol Device:Q_Photo_NPN
- added R7: 20K, Resistor_SMD:R_0201_0603Metric, symbol OSO-SWAT-A1-05-eagle-import:RESISTOR_0603MP
Connections:
- net VCC: now also R7.1
- net A1_SCK renamed LIGHTSENSE
- net LIGHTSENSE: now also Q2.1 (C), R7.2
- net A2_MOSI renamed ~{LS_ENABLE}
- net ~{LS_ENABLE}: now also Q2.2 (E)
- no-connect marks 10 -> 8
